File: Gyrocam BNO055 v2/GyroCam BNO055_v2.brd (EAGLE design)
At the start: 97 x 67 mm, 24 parts, among them IC1 STM32G070KBT6

Commit message: Add files via upload
Parts:
- moved C15 14.2 mm to (21.7, 39.3)
- moved C9 14.2 mm to (28.9, 36.4)
- moved JP1 14.2 mm to (40.6, 24.1)
- moved R1 14.2 mm to (32.4, 32.9)
- moved R2 14.2 mm to (34.7, 32.9)
- moved R6 14.2 mm to (15.8, 38.8)
- moved C16 14.2 mm to (28.8, 14.9)
- moved LED1 14.2 mm to (32.4, 37.5)
- moved R4 14.2 mm to (36.0, 16.6)
- moved U$3 14.2 mm to (22.9, 14.0)
- moved C10 14.2 mm to (28.6, 31.0)
- moved C2 14.2 mm to (25.8, 10.3)
- moved IC1 14.2 mm to (30.5, 21.6)
- moved LEDB 14.2 mm to (17.3, 40.6)
- moved PS1 14.2 mm to (28.3, 33.9)
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Routing:
- net GND: track 18.2 -> 19.3 mm
Other:
- board size 97 x 67 mm -> 57.6 x 50.5 mm
